Commit message: Motion Planner dev for jrnl

File: motion_planner/drake/manipulation/models/jaco_description/urdf/j2s7s300.urdf (robot description, URDF)
Before this commit: robot j2s7s300, 16 links, 15 joints
Links:
- link base: geometry collision sphere radius=0; visual sphere radius=0
- link j2s7s300_end_effector: geometry collision sphere radius=0; visual sphere radius=0
Joints:
- joint j2s7s300_joint_1: limit lower=-6.28318530718 upper=6.28318530718 effort=2000 velocity=1 -> lower=-174.532925 upper=174.532925 effort=2000 velocity=1
- joint j2s7s300_joint_3: limit lower=-6.28318530718 upper=6.28318530718 effort=2000 velocity=1 -> lower=-174.532925 upper=174.532925 effort=2000 velocity=1
- joint j2s7s300_joint_5: limit lower=-6.28318530718 upper=6.28318530718 effort=2000 velocity=1 -> lower=-174.532925 upper=174.532925 effort=2000 velocity=1
- joint j2s7s300_joint_7: limit lower=-6.28318530718 upper=6.28318530718 effort=2000 velocity=1 -> lower=-174.532925 upper=174.532925 effort=2000 velocity=1

File: motion_planner/drake/safe-nav-loco/model/cart.urdf (robot description, URDF)
Before this commit: robot locobot, 25 links, 24 joints
Joints:
- joint base_joint: origin xyz=-9 0 -0.7 rpy=0 0 -0.5 -> xyz=0 0 0 rpy=0 0 -0.5

File: motion_planner/drake/safe-nav-loco/model/cart1.urdf (robot description, URDF)
Before this commit: robot locobot, 25 links, 24 joints
Joints:
- joint base_joint: origin xyz=-3 -3.5 -0.7 rpy=0 0 1.57 -> xyz=0 0 0 rpy=0 0 0
